File: breadboard_6_SOT363/breadboard_6_SOT363.sch (KiCad schematic (older format))
At the start: 2 parts

Commit message: * small updates
Parts:
- added U? (x3): 74LVC1G98, symbol 74LVC1G98
Changed lines of the file:
@@
 LIBS:SquantorProto
 LIBS:SquantorConnectors
+LIBS:SquantorNxp
+LIBS:breadboard_6_SOT363-cache
 EELAYER 25 0
 EELAYER END
@@
 Wire Wire Line
 	3650 2800 3700 2800
+$Comp
+L 74LVC1G98 U?
+U 1 1 596FC94A
+P 2650 2000
+F 0 "U?" H 2650 2250 60  0000 C CNN
+F 1 "74LVC1G98" H 2650 1750 60  0000 C CNN
+F 2 "" H 2650 2000 60  0001 C CNN
+F 3 "" H 2650 2000 60  0001 C CNN
+	1    2650 2000
+	1    0    0    -1
+$EndComp
+$Comp
+L 74LVC1G98 U?
+U 1 1 596FC98B
+P 2650 2600
+F 0 "U?" H 2650 2850 60  0000 C CNN
+F 1 "74LVC1G98" H 2650 2350 60  0000 C CNN
+F 2 "" H 2650 2600 60  0001 C CNN
+F 3 "" H 2650 2600 60  0001 C CNN
+	1    2650 2600
+	1    0    0    -1
+$EndComp
+$Comp
+L 74LVC1G98 U?
+U 1 1 596FC9C8
+P 2650 3200
+F 0 "U?" H 2650 3450 60  0000 C CNN
+F 1 "74LVC1G98" H 2650 2950 60  0000 C CNN
+F 2 "" H 2650 3200 60  0001 C CNN
+F 3 "" H 2650 3200 60  0001 C CNN
+	1    2650 3200
+	1    0    0    -1
+$EndComp
 $EndSCHEMATC
